File: pcb/stm32g4-usbd-devboard/stm32g4-usbd-devboard.kicad_sch (KiCad schematic)
At the start: 29 parts, among them J1 USB_B_Mini, J2 PIN H 6P, J3 LEFT, J4 RIGHT, U1 USBLC6-2SC6, U2 MCP1700-3302E, U3 STM32G431KBTx, Y1 24MHz

Commit message: pcb: *: new revision: 20250412
Parts:
- C4, R1: now not fitted
- J2: Descr SWD -> (none); STM32_PIN2 (none) -> A14; STM32_PIN4 (none) -> A13; STM32_PIN6 (none) -> B3
- J5: renamed from JP2; symbol Jumper:Jumper_2_Open -> Connector_Generic:Conn_01x02
Other:
- moved on the sheet: C10, C11, C5, C6, C7, C8, C9, U3, Y1
