File: pcb/stm32c0-usbd-devboard/stm32c0-usbd-devboard.kicad_pcb (KiCad board)
At the start: 2 copper layers, 23.1 x 56.9 mm, 26 parts, among them J1 USB_B_Mini, J2 PIN H 5P, J3 LEFT, J4 RIGHT, U1 USBLC6-2SC6, U2 MCP1700-3302E, U3 STM32C071K8T6, Y1 8MHz

Commit message: pcb: c0: fix crystal frequency
no physical layer changes, no revision bump.
Parts:
- Y1: value 8MHz -> 48MHz
Changed lines of the file:
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@@
 			)
 		)
-		(property "Value" "8MHz"
+		(property "Value" "48MHz"
 			(at 2.44 3.525 90)
 			(layer "F.Fab")
